File: mullet-pcb.sch (KiCad schematic (older format))
At the start: 183 parts, among them SW1 KEYSW, SW10 KEYSW, SW11 KEYSW, SW12 KEYSW, SW13 KEYSW, SW14 KEYSW, SW15 KEYSW, SW16 KEYSW, SW17 KEYSW, SW18 KEYSW, SW19 KEYSW, SW2 KEYSW, SW20 KEYSW, SW21 KEYSW, SW22 KEYSW, SW23 KEYSW, SW24 KEYSW, SW25 KEYSW, SW26 KEYSW, SW27 KEYSW, SW28 KEYSW, SW29 KEYSW, SW3 KEYSW, SW30 KEYSW, SW31 KEYSW, SW32 KEYSW, SW33 KEYSW, SW34 KEYSW, SW35 KEYSW, SW36 KEYSW, SW37 KEYSW, SW38 KEYSW, SW39 KEYSW, SW4 KEYSW, SW40 KEYSW, SW41 KEYSW, SW42 KEYSW, SW43 KEYSW, SW44 KEYSW, SW45 KEYSW, SW46 KEYSW, SW47 KEYSW, SW48 KEYSW, SW49 KEYSW, SW5 KEYSW, SW50 KEYSW, SW51 KEYSW, SW52 KEYSW, SW53 KEYSW, SW54 KEYSW, SW55 KEYSW, SW56 KEYSW, SW57 KEYSW, SW58 KEYSW, SW59 KEYSW, SW6 KEYSW, SW60 KEYSW, SW61 KEYSW, SW62 KEYSW, SW63 KEYSW, SW64 KEYSW, SW65 KEYSW, SW66 KEYSW, SW67 KEYSW, SW7 KEYSW, SW8 KEYSW, SW9 KEYSW, U1 ATMEGA32U4, U2 PRTR5V0U2X, X1 XTAL_GND

Commit message: clean up schematic
Parts:
- USB1: symbol Type-C:HRO-TYPE-C-31-M-12 -> mullet-pcb-rescue:HRO-TYPE-C-31-M-12-Type-C
Changed lines of the file:
@@
 EESchema Schematic File Version 4
 LIBS:mullet-pcb-cache
-EELAYER 26 0
+EELAYER 29 0
 EELAYER END
 $Descr A4 11693 8268
@@
 D+
 $Comp
-L Type-C:HRO-TYPE-C-31-M-12 USB1
+L mullet-pcb-rescue:HRO-TYPE-C-31-M-12-Type-C USB1
 U 1 1 5C71D73F
 P 1350 4850
